File: kicad/main20220103/main20220103.kicad_pcb (KiCad board)
At the start: 2 copper layers, 170 x 141.9 mm, 74 parts, among them J1 Power IN, J10 drib-kick, J11 LINE, J12 Serial3/Vision, J13 Serial2/IMU, J14 MD1, J15 MD2, J16 Drib-Kick, J17 USB_B_Micro, J18 USB-micro-b, J2 XBee, J26 Trimmer, J3 I2C_ToF, J4 I2C_OLED, J5 raspi-power, J6 MD1, J7 MD2, J8 MD3, J9 MD4, Q1 AO3400A, SW1 Reset, SW2 PROG, SW4 SW_SPST, SW5 GOAL, SW6 START, U1 OKL-T_3-W12N-C, U2 74HC32, U3 74HC04, U4 Teensy3.5

Commit message: pcb
Parts:
- removed the J17 at (143.7, 143.0)
- added J18: MD3, Connector_JST:JST_XH_B2B-XH-A_1x02_P2.50mm_Vertical, F.Cu at (121.0, 95.2)
- added J19: MD4, Connector_JST:JST_XH_B2B-XH-A_1x02_P2.50mm_Vertical, F.Cu at (109.8, 56.2)
- added J9: micro-b_out, Connector_PinHeader_2.54mm:PinHeader_1x05_P2.54mm_Vertical, F.Cu at (129.9, 125.0)
- added Q2: AO3401A, Package_TO_SOT_SMD:SOT-23, F.Cu at (106.0, 128.0)
- added R10: 47k, Resistor_SMD:R_0603_1608Metric_Pad0.98x0.95mm_HandSolder, F.Cu at (127.0, 152.0)
- added R18: 10k, Resistor_SMD:R_0603_1608Metric_Pad0.98x0.95mm_HandSolder, F.Cu at (104.0, 132.0)
- added SW3: SET, Button_Switch_THT:SW_PUSH_6mm, F.Cu at (116.8, 152.8)
- J1: renamed from J7; footprint 0.main.robot:JSTB4B-ZR -> 0.main.robot:JSTS4B-ZRLFSN; moved to F.Cu
- J10: renamed from J18; value USB-micro-b -> micro-b_in
- J11: renamed from J3; footprint 0.main.robot:JSTB4B-ZR -> 0.main.robot:JSTS4B-ZRLFSN; moved to F.Cu
- J15: renamed from J11; footprint 0.main.robot:JSTB8B-ZR -> 0.main.robot:JSTS8B-ZRLFSN; moved to F.Cu
- J16: renamed from J14; moved to F.Cu
- J17: renamed from J15; moved to F.Cu
- J2: renamed from J9; footprint 0.main.robot:JSTB4B-ZR -> 0.main.robot:JSTS4B-ZRLFSN; moved to F.Cu
- J21: renamed from J26; moved to F.Cu
- J3: renamed from J8; footprint 0.main.robot:JSTB4B-ZR -> 0.main.robot:JSTS4B-ZRLFSN; moved to F.Cu
- J4: renamed from J6; footprint 0.main.robot:JSTB4B-ZR -> 0.main.robot:JSTS4B-ZRLFSN; moved to F.Cu
- J5: renamed from J2; moved to B.Cu
- J8: renamed from J13; footprint Connector_PinSocket_2.54mm:PinSocket_1x04_P2.54mm_Vertical -> Connector_PinSocket_2.54mm:PinSocket_1x05_P2.54mm_Vertical
- Q1: footprint Package_TO_SOT_SMD:SOT-23_Handsoldering -> Package_TO_SOT_SMD:SOT-23
- moved SW1 113.4 mm to (53.0, 80.0), turned to -90 degrees
- moved C4 106.2 mm to (53.0, 86.0), turned to -90 degrees
- moved C5 97.6 mm to (53.0, 93.0), turned to -90 degrees
- moved SW2 93.4 mm to (53.0, 100.0), turned to -90 degrees
- moved R2 86.8 mm to (182.0, 99.0), turned to 180 degrees
- moved R1 75.5 mm to (174.0, 99.0), turned to 180 degrees
- moved U3 69.9 mm to (85.0, 93.0), turned to 90 degrees
- moved R13 69.3 mm to (139.0, 33.0), turned to 0 degrees
- moved R3 67.5 mm to (179.0, 76.0), turned to 180 degrees
- moved R7 66.0 mm to (175.0, 76.0), turned to 180 degrees
- moved R6 65.0 mm to (171.0, 76.0), turned to 180 degrees
- moved Q1 63.8 mm to (101.0, 128.0), turned to 0 degrees
- moved D2 62.6 mm to (175.0, 89.1), turned to 90 degrees
- moved R14 61.8 mm to (139.0, 37.0), turned to 0 degrees
- moved R17 56.6 mm to (135.0, 37.0), turned to 0 degrees
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- renumbered C5 to C4, C4 to C5, D2 to D1, D1 to D2, D8 to D3, D6 to D4, D7 to D5, D9 to D6, D10 to D7, J4 to J12, J10 to J13, J1 to J14, J16 to J20, J12 to J6, J5 to J7, R3 to R1, R6 to R11, R7 to R12, R10 to R13, R11 to R14, R23 to R16, R12 to R17, R28 to R19, R4 to R2, R24 to R20, R25 to R21, R26 to R22, R27 to R23, R29 to R24, R30 to R25, R31 to R26, R32 to R27, R2 to R3, R21 to R4, R22 to R5, R1 to R6, R5 to R7, RV2 to RV1, RV3 to RV2, RV4 to RV3, RV5 to RV4, RV6 to RV5, SW2 to SW1, SW1 to SW2, U4 to U2, U2 to U3, U3 to U4
Connections:
- J15 pad 4: +5V -> Net-(J15-Pad4)
- J15 pad 8: Net-(J11-Pad8) -> GND
- J8 pad 1: Net-(J13-Pad1) (its old number) -> Net-(J8-Pad1)
- J8 pad 2: +5V -> Net-(J8-Pad2)
- J8 pad 3: Net-(J13-Pad3) (its old number) -> +5V
- J8 pad 4: GND -> Net-(J8-Pad4)
- Q1 pad 3: Net-(J11-Pad8) -> Net-(Q1-Pad3)
- R24 pad 1: +5V -> +3V3
- R25 pad 1: +5V -> +3V3
- R5 pad 2: Net-(J13-Pad3) (its old number) -> Net-(J8-Pad4)
- U2 pad 12: Net-(J13-Pad1) (its old number) -> Net-(J8-Pad2)
Routing:
- net GND: track 0.00 -> 25.2 mm, vias 0 -> 1
Other:
- board size 170 x 141.9 mm -> 170 x 141.4 mm
