File: kicad/main20220213/main20220213.kicad_pcb (KiCad board)
At the start: 2 copper layers, 170 x 141.4 mm, 80 parts, among them J1 MD2, J10 micro-b_in, J11 I2C_ToF, J12 I2C_OLED, J13 drib-kick, J14 Power IN, J15 LINE, J16 MD1, J17 MD2, J18 MD3, J19 MD4, J2 MD4, J20 Drib-Kick, J21 Trimmer, J3 MD3, J4 MD1, J5 XBee, J6 Serial3/Vision, J7 raspi-power, J8 Serial2/IMU, J9 micro-b_out, Q1 AO3400A, Q2 AO3401A, SW1 PROG, SW2 Reset, SW3 SET, SW4 SW_SPST, SW5 GOAL, SW6 START, U1 OKL-T_3-W12N-C, U2 Teensy3.5, U3 74HC32, U4 74HC04

Commit message: pcb
Parts:
- C2, R11, R12, R8, R9, U3, U4: moved to B.Cu
- moved R8 99.2 mm to (55.0, 71.0), turned to 180 degrees
- moved U4 94.8 mm to (85.0, 102.0), turned to 180 degrees
- moved R9 82.9 mm to (55.0, 109.0), turned to 180 degrees
- moved R16 42.0 mm to (112.0, 57.0)
- moved R15 33.2 mm to (114.0, 62.0)
- moved U3 25.0 mm to (85.0, 80.0), turned to 180 degrees
- moved Q2 22.1 mm to (100.0, 96.0)
- moved R17 18.7 mm to (117.0, 66.0)
- moved Q1 16.6 mm to (100.0, 85.0)
- moved R13 16.2 mm to (122.0, 74.0)
- moved R11 12.2 mm to (135.0, 125.0), turned to 180 degrees
- moved R7 12.0 mm to (173.0, 76.0), turned to 90 degrees
- moved R12 12.0 mm to (141.0, 125.0), turned to 180 degrees
- moved J21 11.0 mm to (131.0, 45.0)
- moved R6 10.0 mm to (165.0, 78.0), turned to 0 degrees
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Routing:
- net +5V: track 0.00 -> 72.5 mm
- net GND: track 268.6 -> 198.6 mm, vias 0 -> 1
