File: kicad/main20220213/main20220213.kicad_sch (KiCad schematic)
At the start: 64 parts, among them J1 MD2, J10 micro-b_in, J11 I2C_ToF, J12 I2C_OLED, J13 drib-kick, J14 Power IN, J15 LINE, J16 MD1, J17 MD2, J18 MD3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

Commit message: pcb
Other:
- moved on the sheet: D3, F1, J10, J14, J16, J17, J18, J19, J20, J7, J9, R19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
