File: kicad/kick-drib/kick-drib.kicad_pcb (KiCad board)
At the start: 2 copper layers, 69.2 x 61.6 mm, 22 parts, among them J1 drib-kick, J2 Conn_01x03, J3 DribblerMotor, J4 drib-kick_POWER, J5 Kicker1, K1 G5V-1/12V, Q1 NP52N06SLG, U1 TLP152, U2 TLP152, U3 XL6009/HW-432

Commit message: pcb
Routing:
- added copper zone on B.Cu, net GND
- added copper zone on F.Cu, net GND
Other:
- outline, holes or cut-outs redrawn

Commit message: iicad
Parts:
- added G***: LOGO, LOGO, F.Cu at (55.0, 99.0)
- turned U3 to 180 degrees
Connections:
- C1 pad 1: +15V -> Net-(J4-Pad1)
- D1 pad 1: +15V -> Net-(J4-Pad1)
- J3 pad 1: +15V -> Net-(J4-Pad1)
- J4 pad 1: +15V -> Net-(J4-Pad1)
- U1 pad 6: +15V -> Net-(J4-Pad1)
Routing:
- net Net-(J4-Pad1): track 0.00 -> 107.0 mm, vias 0 -> 2
- net +15V: track 134.8 -> 49.1 mm, vias 4 -> 2
- net Net-(R3-Pad2): track 70.0 -> 29.5 mm
- net GND: track 164.0 -> 140.7 mm, vias 3 -> 0
- net Net-(R2-Pad1): track 27.2 -> 13.7 mm
- net Net-(J2-Pad1): track 29.0 -> 36.6 mm
- net Net-(R1-Pad1): track 2.95 -> 10.4 mm
- net Net-(J1-Pad4): track 76.8 -> 69.5 mm
- net Net-(J1-Pad3): track 57.5 -> 50.7 mm
- net Net-(D1-Pad2): track 27.8 -> 33.4 mm
- net Net-(C3-Pad1): track 60.2 -> 55.6 mm
- net Net-(Q1-Pad1): track 12.0 -> 14.0 mm, vias 2 -> 0
- net Net-(J2-Pad2): track 37.4 -> 38.4 mm
- net Net-(J1-Pad1): track 21.3 -> 21.9 mm, vias 1 -> 0
- net Net-(J5-Pad1): track 33.8 -> 34.0 mm, vias 0 -> 1
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Other:
- board text added: "Kick-Drib Feb.2022 by A.Saeki"
