File: kicad/kick-drib/kick-drib.kicad_sch (KiCad schematic)
At the start: 22 parts, among them J1 drib-kick, J2 Conn_01x03, J3 DribblerMotor, J4 drib-kick_POWER, J5 Kicker1, K1 G5V-1/12V, Q1 NP52N06SLG, U1 TLP152, U2 TLP152, U3 XL6009/HW-432

Commit message: iicad
Connections:
- net +15V: no longer C1.1, D1.1 (K), J3.1 (Pin_1), J4.1 (Pin_1), U1.6 (VCC)
- new net: C1.1, D1.1 (K), J3.1 (Pin_1), J4.1 (Pin_1), U1.6 (VCC)
Other:
- moved on the sheet: J4
Changed lines of the file:
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@@
   (junction (at 220.98 144.78) (diameter 0) (color 0 0 0 0)
   )
-  (junction (at 199.39 144.78) (diameter 0) (color 0 0 0 0)
-  )
   (junction (at 133.35 57.15) (diameter 0) (color 0 0 0 0)
   )
@@
   (junction (at 115.57 44.45) (diameter 0) (color 0 0 0 0)
   )
-  (junction (at 228.6 59.69) (diameter 0) (color 0 0 0 0)
-  )
   (junction (at 120.65 144.78) (diameter 0) (color 0 0 0 0)
   )
@@
   (junction (at 100.33 173.99) (diameter 0) (color 0 0 0 0)
   )
-  (junction (at 233.68 67.31) (diameter 0) (color 0 0 0 0)
-  )
-  (junction (at 199.39 123.19) (diameter 0) (color 0 0 0 0)
+  (junction (at 173.99 71.12) (diameter 0) (color 0 0 0 0)
   )
   (junction (at 133.35 76.2) (diameter 0) (color 0 0 0 0)
@@
     (stroke (width 0) (type default) (color 0 0 0 0))
   )
-  (wire (pts (xy 167.64 63.5) (xy 170.18 63.5))
+  (wire (pts (xy 167.64 63.5) (xy 176.53 63.5))
     (stroke (width 0) (type default) (color 0 0 0 0))
   )
@@
     (stroke (width 0) (type default) (color 0 0 0 0))
   )
-  (wire (pts (xy 236.22 64.77) (xy 228.6 64.77))
-    (stroke (width 0) (type default) (color 0 0 0 0))
-  )
   (wire (pts (xy 175.26 144.78) (xy 175.26 196.85))
     (stroke (width 0) (type default) (color 0 0 0 0))
@@
     (stroke (width 0) (type default) (color 0 0 0 0))
   )
-  (wire (pts (xy 228.6 59.69) (xy 236.22 59.69))
-    (stroke (width 0) (type default) (color 0 0 0 0))
-  )
   (wire (pts (xy 133.35 57.15) (xy 177.8 57.15))
     (stroke (width 0) (type default) (color 0 0 0 0))
@@
     (stroke (width 0) (type default) (color 0 0 0 0))
   )
-  (wire (pts (xy 228.6 64.77) (xy 228.6 59.69))
-    (stroke (width 0) (type default) (color 0 0 0 0))
-  )
-  (wire (pts (xy 184.15 144.78) (xy 199.39 144.78))
+  (wire (pts (xy 184.15 144.78) (xy 220.98 144.78))
     (stroke (width 0) (type default) (color 0 0 0 0))
   )
@@
     (stroke (width 0) (type default) (color 0 0 0 0))
   )
-  (wire (pts (xy 236.22 62.23) (xy 233.68 62.23))
+  (wire (pts (xy 176.53 66.04) (xy 173.99 66.04))
     (stroke (width 0) (type default) (color 0 0 0 0))
   )
@@
     (stroke (width 0) (type default) (color 0 0 0 0))
   )
-  (wire (pts (xy 184.15 123.19) (xy 199.39 123.19))
+  (wire (pts (xy 184.15 123.19) (xy 207.01 123.19))
     (stroke (width 0) (type default) (color 0 0 0 0))
   )
@@
     (stroke (width 0) (type default) (color 0 0 0 0))
   )
-  (wire (pts (xy 199.39 144.78) (xy 220.98 144.78))
-    (stroke (width 0) (type default) (color 0 0 0 0))
-  )
   (wire (pts (xy 115.57 44.45) (xy 133.35 44.45))
     (stroke (width 0) (type default) (color 0 0 0 0))
@@
     (stroke (width 0) (type default) (color 0 0 0 0))
   )
-  (wire (pts (xy 199.39 123.19) (xy 199.39 133.35))
-    (stroke (width 0) (type default) (color 0 0 0 0))
-  )
   (wire (pts (xy 220.98 144.78) (xy 240.03 144.78))
     (stroke (width 0) (type default) (color 0 0 0 0))
@@
     (stroke (width 0) (type default) (color 0 0 0 0))
   )
-  (wire (pts (xy 199.39 135.89) (xy 199.39 144.78))
-    (stroke (width 0) (type default) (color 0 0 0 0))
-  )
-  (wire (pts (xy 233.68 62.23) (xy 233.68 67.31))
-    (stroke (width 0) (type default) (color 0 0 0 0))
-  )
-  (wire (pts (xy 199.39 123.19) (xy 207.01 123.19))
+  (wire (pts (xy 173.99 66.04) (xy 173.99 71.12))
     (stroke (width 0) (type default) (color 0 0 0 0))
   )
@@
     (stroke (width 0) (type default) (color 0 0 0 0))
   )
-  (wire (pts (xy 231.14 67.31) (xy 233.68 67.31))
+  (wire (pts (xy 171.45 71.12) (xy 173.99 71.12))
     (stroke (width 0) (type default) (color 0 0 0 0))
   )
@@
     (stroke (width 0) (type default) (color 0 0 0 0))
   )
-  (wire (pts (xy 233.68 67.31) (xy 236.22 67.31))
-    (stroke (width 0) (type default) (color 0 0 0 0))
-  )
-  (wire (pts (xy 228.6 57.15) (xy 228.6 59.69))
+  (wire (pts (xy 173.99 71.12) (xy 176.53 71.12))
     (stroke (width 0) (type default) (color 0 0 0 0))
   )
@@
     (pin "2")
   )
-  (symbol (lib_id "Connector_Generic:Conn_01x04") (at 241.3 62.23 0) (unit 1)
-    (in_bom yes) (on_board yes)
-    (property "Reference" "J4" (id 0) (at 239.2172 54.1782 0))
-    (property "Value" "drib-kick_POWER" (id 1) (at 239.2172 56.4896 0))
-    (property "Footprint" "Connector_PinHeader_2.54mm:PinHeader_1x04_P2.54mm_Vertical" (id 2) (at 241.3 62.23 0)
-      (effects (font (size 1.27 1.27)) hide)
-    )
-    (property "Datasheet" "~" (id 3) (at 241.3 62.23 0)
+  (symbol (lib_id "Connector_Generic:Conn_01x04") (at 181.61 66.04 0) (unit 1)
+    (in_bom yes) (on_board yes)
+    (property "Reference" "J4" (id 0) (at 179.5272 57.9882 0))
+    (property "Value" "drib-kick_POWER" (id 1) (at 179.5272 60.2996 0))
+    (property "Footprint" "Connector_PinHeader_2.54mm:PinHeader_1x04_P2.54mm_Vertical" (id 2) (at 181.61 66.04 0)
+      (effects (font (size 1.27 1.27)) hide)
+    )
+    (property "Datasheet" "~" (id 3) (at 181.61 66.04 0)
       (effects (font (size 1.27 1.27)) hide)
     )
@@
     (pin "2")
   )
-  (symbol (lib_id "power:+15V") (at 228.6 57.15 0) (unit 1)
-    (in_bom yes) (on_board yes)
-    (property "Reference" "#PWR0108" (id 0) (at 228.6 60.96 0)
-      (effects (font (size 1.27 1.27)) hide)
-    )
-    (property "Value" "+15V" (id 1) (at 228.981 52.7558 0))
-    (property "Footprint" "" (id 2) (at 228.6 57.15 0)
-      (effects (font (size 1.27 1.27)) hide)
-    )
-    (property "Datasheet" "" (id 3) (at 228.6 57.15 0)
-      (effects (font (size 1.27 1.27)) hide)
-    )
-    (pin "1")
-  )
-  (symbol (lib_id "power:GND") (at 231.14 67.31 270) (unit 1)
-    (in_bom yes) (on_board yes)
-    (property "Reference" "#PWR0109" (id 0) (at 224.79 67.31 0)
-      (effects (font (size 1.27 1.27)) hide)
-    )
-    (property "Value" "GND" (id 1) (at 226.7458 67.437 0))
-    (property "Footprint" "" (id 2) (at 231.14 67.31 0)
-      (effects (font (size 1.27 1.27)) hide)
-    )
-    (property "Datasheet" "" (id 3) (at 231.14 67.31 0)
+  (symbol (lib_id "power:+15V") (at 176.53 68.58 90) (unit 1)
+    (in_bom yes) (on_board yes)
+    (property "Reference" "#PWR0108" (id 0) (at 180.34 68.58 0)
+      (effects (font (size 1.27 1.27)) hide)
+    )
+    (property "Value" "+15V" (id 1) (at 172.1358 68.199 0))
+    (property "Footprint" "" (id 2) (at 176.53 68.58 0)
+      (effects (font (size 1.27 1.27)) hide)
+    )
+    (property "Datasheet" "" (id 3) (at 176.53 68.58 0)
+      (effects (font (size 1.27 1.27)) hide)
+    )
+    (pin "1")
+  )
+  (symbol (lib_id "power:GND") (at 171.45 71.12 270) (unit 1)
+    (in_bom yes) (on_board yes)
+    (property "Reference" "#PWR0109" (id 0) (at 165.1 71.12 0)
+      (effects (font (size 1.27 1.27)) hide)
+    )
+    (property "Value" "GND" (id 1) (at 167.0558 71.247 0))
+    (property "Footprint" "" (id 2) (at 171.45 71.12 0)
+      (effects (font (size 1.27 1.27)) hide)
+    )
+    (property "Datasheet" "" (id 3) (at 171.45 71.12 0)
       (effects (font (size 1.27 1.27)) hide)
     )
@@
     (pin "2")
   )
-  (symbol (lib_id "power:+15V") (at 170.18 63.5 270) (unit 1)
-    (in_bom yes) (on_board yes)
-    (property "Reference" "#PWR0102" (id 0) (at 166.37 63.5 0)
-      (effects (font (size 1.27 1.27)) hide)
-    )
-    (property "Value" "+15V" (id 1) (at 174.5742 63.881 0))
-    (property "Footprint" "" (id 2) (at 170.18 63.5 0)
-      (effects (font (size 1.27 1.27)) hide)
-    )
-    (property "Datasheet" "" (id 3) (at 170.18 63.5 0)
-      (effects (font (size 1.27 1.27)) hide)
-    )
-    (pin "1")
-  )
   (sheet_instances
     (path "/" (page "1"))
@@
       (reference "#PWR0101") (unit 1) (value "GND") (footprint "")
     )
-    (path "/ff72b64a-8dc3-4b06-9bdf-8a29a3f3b4ef"
-      (reference "#PWR0102") (unit 1) (value "+15V") (footprint "")
-    )
     (path "/c6ba4aa1-16a1-48ea-9b03-bef98e18820d"
