File: kicad/xbee-gyro20220207/xbee-gyro20220207.kicad_sch (KiCad schematic)
At the start: 17 parts, among them J1 IMU_in, J2 IMU, J3 XBee, SW1 Reset, U1 XBEE-S2C, U2 XC6216D_SOT89

Commit message: pcb
Changed lines of the file:
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@@
     (pin "9")
-  )
-  (symbol (lib_id "power:+5V") (at 102.87 24.13 0) (unit 1)
-    (in_bom yes) (on_board yes)
-    (property "Reference" "#PWR0105" (id 0) (at 102.87 27.94 0)
-      (effects (font (size 1.27 1.27)) hide)
-    )
-    (property "Value" "+5V" (id 1) (at 103.251 19.7358 0))
-    (property "Footprint" "" (id 2) (at 102.87 24.13 0)
-      (effects (font (size 1.27 1.27)) hide)
-    )
-    (property "Datasheet" "" (id 3) (at 102.87 24.13 0)
-      (effects (font (size 1.27 1.27)) hide)
-    )
-    (pin "1")
   )
   (symbol (lib_id "Device:LED") (at 215.9 148.59 90) (unit 1)
@@
       (reference "#PWR0104") (unit 1) (value "GND") (footprint "")
     )
-    (path "/d427b096-2104-4cac-9d5d-d2195401989e"
-      (reference "#PWR0105") (unit 1) (value "+5V") (footprint "")
-    )
     (path "/a231a5c3-b8cd-4dcd-ac6c-04c40c185a50"

Commit message: no message
Parts:
- J1: footprint Connector_PinSocket_2.54mm:PinSocket_1x05_P2.54mm_Vertical -> Connector_PinHeader_1.27mm:PinHeader_1x05_P1.27mm_Vertical
Changed lines of the file:
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@@
       (effects (font (size 1.27 1.27)) (justify right))
     )
-    (property "Footprint" "Connector_PinSocket_2.54mm:PinSocket_1x05_P2.54mm_Vertical" (id 2) (at 217.17 78.74 0)
+    (property "Footprint" "Connector_PinHeader_1.27mm:PinHeader_1x05_P1.27mm_Vertical" (id 2) (at 217.17 78.74 0)
       (effects (font (size 1.27 1.27)) hide)
     )
@@
     )
     (path "/30d4a5b8-34e9-412f-9d1a-e616a8a28215"
-      (reference "J1") (unit 1) (value "IMU_in") (footprint "Connector_PinSocket_2.54mm:PinSocket_1x05_P2.54mm_Vertical")
+      (reference "J1") (unit 1) (value "IMU_in") (footprint "Connector_PinHeader_1.27mm:PinHeader_1x05_P1.27mm_Vertical")
     )
     (path "/0bf7f675-adbe-42d7-8d1e-a9414fad6301"
